File: PCB/LED-Brillen-Adapter-PCB.kicad_pcb (KiCad board)
At the start: 2 copper layers, 28.7 x 28.8 mm, 10 parts, among them J1 Conn_01x07_Pin, J2 Conn_01x07_Pin, J3 Conn_01x03_Pin, J4 Conn_01x02, J5 Conn_01x02, SW1 SW_DIP_x01, SW2 SW_Push

Commit message: Added rev. 3
Parts:
- removed SW: ~, Library-MSS-2336-DTE:MSS-2336
- added SW3: ~, Library-MSS-2336-DTE:MSS-2336, F.Cu at (220.0, 96.1)
- R1, R2: footprint Resistor_THT:R_Axial_DIN0204_L3.6mm_D1.6mm_P2.54mm_Vertical -> Resistor_THT:R_Axial_DIN0204_L3.6mm_D1.6mm_P5.08mm_Horizontal
- moved SW1 70.0 mm to (216.0, 95.8), turned to 90 degrees
- moved J1 60.9 mm to (247.1, 98.0)
- moved J2 60.9 mm to (247.1, 80.2)
- moved J4 60.9 mm to (239.7, 83.8)
- moved R2 60.9 mm to (227.5, 81.0), turned to -90 degrees
- moved R1 59.1 mm to (225.0, 86.0), turned to 90 degrees
- moved J5 57.3 mm to (203.8, 88.0), turned to -90 degrees
- moved J3 47.0 mm to (207.8, 86.7)
- moved SW2 41.2 mm to (215.2, 81.5), turned to 0 degrees
Routing:
- net /Battery-Measurement: track 27.5 -> 17.8 mm
- net GND (Battery): track 38.2 -> 44.6 mm
- net Net-(J5-Pin_1): track 8.17 -> 14.2 mm
- net VCC (Stripe): track 16.9 -> 21.7 mm
- net /LEDS: track 40.5 -> 42.6 mm
- net GND (ESP): track 0.00 -> 1.89 mm, vias 36 -> 40
- net /BTN: track 28.6 -> 26.9 mm
- net 3,7V (BAT): track 33.5 -> 34.8 mm
- net 5V (USB): track 28.6 -> 28.0 mm
- net (no net): vias 1 -> 0
Other:
- board size 28.7 x 28.8 mm -> 50 x 21.5 mm
- board text added: "AN"
- board text added: "AUS"
- board text added: "DATA"
- board text added: "LED-Brillen Adapter Rev. 3 Noah Albers ARTandTECH.space / Projektlabor"
- board text added: "LED: GPIO3 BTN: GPIO2"
- board text removed: "Battery"
- board text removed: "Button"
- board text removed: "Data"
- board text removed: "Mode Switch"
- board text removed: "Off"
- board text removed: "On"
- board text removed: "On/Off"
