File: PCB/LED-Brillen-Adapter-PCB.kicad_sch (KiCad schematic)
At the start: 10 parts, among them J1 Conn_01x07_Pin, J2 Conn_01x07_Pin, J3 Conn_01x03_Pin, J4 Conn_01x02, J5 Conn_01x02, SW1 SW_DIP_x01, SW2 SW_Push

Commit message: Added rev. 3
Parts:
- R1, R2: footprint Resistor_THT:R_Axial_DIN0204_L3.6mm_D1.6mm_P2.54mm_Vertical -> Resistor_THT:R_Axial_DIN0204_L3.6mm_D1.6mm_P5.08mm_Horizontal
- renumbered SW to SW3
Changed lines of the file:
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@@
 			)
 		)
-		(property "Footprint" "Resistor_THT:R_Axial_DIN0204_L3.6mm_D1.6mm_P2.54mm_Vertical"
+		(property "Footprint" "Resistor_THT:R_Axial_DIN0204_L3.6mm_D1.6mm_P5.08mm_Horizontal"
 			(at 40.132 26.67 90)
 			(effects
@@
 			)
 		)
-		(property "Footprint" "Resistor_THT:R_Axial_DIN0204_L3.6mm_D1.6mm_P2.54mm_Vertical"
+		(property "Footprint" "Resistor_THT:R_Axial_DIN0204_L3.6mm_D1.6mm_P5.08mm_Horizontal"
 			(at 40.132 36.83 90)
 			(effects
@@
 		(on_board yes)
 		(dnp no)
-		(property "Reference" "SW"
+		(property "Reference" "SW3"
 			(at 62.23 73.914 90)
 			(effects
@@
 			(project "LED-Brillen-Adapter-PCB"
 				(path "/5f322e17-ab81-4770-a746-a25aadfbe2be"
-					(reference "SW")
-					(unit 1)
-				)
+					(reference "SW3")
+					(unit 1)
+				)
